Commit message: Organization, rviz config

File: urdf/robot.urdf (robot description, URDF)
Before this commit: robot DeliveryBot, 6 links, 5 joints
Links:
- link body: geometry collision mesh filename=package://deliverybot/urdf/meshes/body.stl; visual mesh filename=package://deliverybot/urdf/meshes/body.stl
- link castor: geometry collision mesh filename=package://deliverybot/urdf/meshes/castor.stl; visual mesh filename=package://deliverybot/urdf/meshes/castor.stl
- link door: geometry collision mesh filename=package://deliverybot/urdf/meshes/door.stl; visual mesh filename=package://deliverybot/urdf/meshes/door.stl
- link left_wheel: geometry collision mesh filename=package://deliverybot/urdf/meshes/left_wheel.stl; visual mesh filename=package://deliverybot/urdf/meshes/left_wheel.stl
- link right_wheel: geometry collision mesh filename=package://deliverybot/urdf/meshes/right_wheel.stl; visual mesh filename=package://deliverybot/urdf/meshes/right_wheel.stl
