Commit message: changed joint positions of wheels to be consistent with diff

File: urdf/robot.xacro (robot description, xacro)
@@ -1,3 +1,4 @@
-<robot name="DeliveryBot">
+<robot name="DeliveryBot" xmlns:xacro="http://www.ros.org/wiki/xacro">
+    <xacro:include filename="$(find deliverybot)/urdf/robot.gazebo"/>
     <link name="base_link"></link>
     <joint name="base_link_to_base" type="fixed">
@@ -26,12 +27,12 @@
         </collision>
         <inertial>
-            <origin xyz="2.01199e-16 0.0116169 0.135939" rpy="0 0 0"/>
-            <mass value="9.56649" />
-            <inertia ixx="0.270308" ixy="0" ixz="-1.76457e-16" iyy="0.296385" iyz="-0.0146076" izz="0.178823" />
+            <origin xyz="7.95747e-17 0.0121391 0.137455" rpy="0 0 0"/>
+            <mass value="9.21638" />
+            <inertia ixx="0.266181" ixy="-3.31633e-16" ixz="-1.63779e-16" iyy="0.281274" iyz="-0.0141244" izz="0.161564" />
         </inertial>
     </link>
     <link name="left_wheel">
         <visual>
-            <origin xyz="0 -0.1 0.155" rpy="-1.5708 -1.5708 0" />
+            <origin xyz="-0.075 -0.1 0.155" rpy="-1.5708 -1.5708 0" />
             <geometry>
                 <mesh filename="package://deliverybot/urdf/meshes/left_wheel.stl"/>
@@ -42,5 +43,5 @@
         </visual>
         <collision>
-            <origin xyz="0 -0.1 0.155" rpy="-1.5708 -1.5708 0" />
+            <origin xyz="-0.075 -0.1 0.155" rpy="-1.5708 -1.5708 0" />
             <geometry>
                 <mesh filename="package://deliverybot/urdf/meshes/left_wheel.stl"/>
@@ -51,11 +52,11 @@
         </collision>
         <inertial>
-            <origin xyz="-2.28687e-18 0 -0.025" rpy="0 0 0"/>
+            <origin xyz="8.32667e-18 0 -0.025" rpy="0 0 0"/>
             <mass value="1.65248" />
             <inertia ixx="0.00447546" ixy="-1.05108e-18" ixz="0" iyy="0.00826239" iyz="0" izz="0.00447546" />
         </inertial>
     </link>
-    <joint name="body_left_wheel" type="continuous">
-        <origin xyz="-0.155 -0.00273569 0.05" rpy="-3.14159 -1.5708 0" />
+    <joint name="joint_left_wheel" type="continuous">
+        <origin xyz="-0.155 0.0722643 0.05" rpy="3.14159 -1.5708 0" />
         <parent link="body" />
         <child link="left_wheel" />
@@ -66,14 +67,14 @@
     <link name="right_wheel">
         <visual>
-            <origin xyz="0 0.1 0.155" rpy="1.5708 1.5708 0" />
+            <origin xyz="-0.075 -0.1 -0.155" rpy="-1.5708 -1.5708 0" />
             <geometry>
                 <mesh filename="package://deliverybot/urdf/meshes/right_wheel.stl"/>
             </geometry>
-            <material name="right_wheel_material">
+            <material name="left_wheel_material">
                 <color rgba="0.498039 0.498039 0.498039 1.0"/>
             </material>
         </visual>
         <collision>
-            <origin xyz="0 0.1 0.155" rpy="1.5708 1.5708 0" />
+            <origin xyz="-0.075 -0.1 -0.155" rpy="-1.5708 -1.5708 0" />
             <geometry>
                 <mesh filename="package://deliverybot/urdf/meshes/right_wheel.stl"/>
@@ -84,11 +85,11 @@
         </collision>
         <inertial>
-            <origin xyz="-2.28687e-18 0 -0.025" rpy="0 0 0"/>
+            <origin xyz="8.32667e-18 0 -0.025" rpy="0 0 0"/>
             <mass value="1.65248" />
-            <inertia ixx="0.00447546" ixy="1.05108e-18" ixz="0" iyy="0.00826239" iyz="0" izz="0.00447546" />
+            <inertia ixx="0.00447546" ixy="-1.05108e-18" ixz="0" iyy="0.00826239" iyz="0" izz="0.00447546" />
         </inertial>
     </link>
-    <joint name="body_right_wheel" type="continuous">
-        <origin xyz="0.155 -0.00273569 0.05" rpy="-2.77556e-16 -1.5708 0" />
+    <joint name="joint_right_wheel" type="continuous">
+        <origin xyz="0.155 0.0722643 0.05" rpy="3.14159 -1.5708 0" />
         <parent link="body" />
         <child link="right_wheel" />
@@ -122,5 +123,5 @@
         </inertial>
     </link>
-    <joint name="body_castor" type="fixed">
+    <joint name="joint_castor" type="fixed">
         <origin xyz="-5.55112e-17 -0.127736 -0.025" rpy="0 -0 0" />
         <parent link="body" />
@@ -152,8 +153,8 @@
             <origin xyz="-0.000258506 0.145116 -0.145" rpy="0 0 0"/>
             <mass value="0.596718" />
-            <inertia ixx="0.00521211" ixy="1.20185e-47" ixz="2.98715e-05" iyy="0.00816722" iyz="5.06885e-50" izz="0.0129235" />
+            <inertia ixx="0.00521211" ixy="0" ixz="2.98715e-05" iyy="0.00816722" iyz="0" izz="0.0129235" />
         </inertial>
     </link>
-    <joint name="body_door" type="revolute">
+    <joint name="joint_door" type="revolute">
         <origin xyz="0.145 -0.129736 0.155" rpy="-3.14159 -1.5708 0" />
         <parent link="body" />
@@ -163,3 +164,36 @@
         <joint_properties friction="0.0"/>
     </joint>
+    <link name="sensor_laser">
+        <visual>
+            <origin xyz="0 -0.125 0.56" rpy="3.14159 -0 0" />
+            <geometry>
+                <mesh filename="package://deliverybot/urdf/meshes/sensor_laser.stl"/>
+            </geometry>
+            <material name="sensor_laser_material">
+                <color rgba="0.34902 0.376471 0.4 1.0"/>
+            </material>
+        </visual>
+        <collision>
+            <origin xyz="0 -0.125 0.56" rpy="3.14159 -0 0" />
+            <geometry>
+                <mesh filename="package://deliverybot/urdf/meshes/sensor_laser.stl"/>
+            </geometry>
+            <material name="sensor_laser_material">
+                <color rgba="0.34902 0.376471 0.4 1.0"/>
+            </material>
+        </collision>
+        <inertial>
+            <origin xyz="3.75509e-19 0 -0.0125" rpy="0 0 0"/>
+            <mass value="0.0516399" />
+            <inertia ixx="1.07583e-05" ixy="0" ixz="0" iyy="1.07583e-05" iyz="0" izz="1.61375e-05" />
+        </inertial>
+    </link>
+    <joint name="joint_laser_sensor" type="fixed">
+        <origin xyz="-5.55112e-17 -0.127736 0.51" rpy="3.14159 -0 0" />
+        <parent link="body" />
+        <child link="sensor_laser" />
+        <axis xyz="0 0 1"/>
+        <limit effort="1" velocity="20" />
+        <joint_properties friction="0.0"/>
+    </joint>
 </robot>
