Commit message: deliverybot_control added but doesn't control gazebo only rviz. Changed directory structure.

File: deliverybot/urdf/robot.xacro (robot description, xacro)
@@ -1,5 +1,6 @@
 <robot name="DeliveryBot" xmlns:xacro="http://www.ros.org/wiki/xacro">
     <xacro:include filename="$(find deliverybot)/urdf/robot.gazebo"/>
-    <link name="base_link"></link>
+    <link name="base_link">
+    </link>
     <joint name="base_link_to_base" type="fixed">
         <parent link="base_link"/>
