Commit message: laser and gmapping synced

File: deliverybot/urdf/dbot_laser.xacro (robot description, xacro)
@@ -6,5 +6,5 @@
         <parent link="base_link"/>
         <child link="body" />
-        <origin rpy="0.0 0 0" xyz="0 0 0"/>
+        <origin xyz="0 0 0" rpy="0 0 3.141" />
     </joint>
     <link name="body">
@@ -59,5 +59,5 @@
     </link>
     <joint name="joint_left_wheel" type="continuous">
-        <origin xyz="-0.155 0.0722643 0.05" rpy="3.14159 -1.5708 0" />
+        <origin xyz="0.155 0.0722643 0.05" rpy="3.14159 -1.5708 0" />
         <parent link="body" />
         <child link="left_wheel" />
@@ -92,5 +92,5 @@
     </link>
     <joint name="joint_right_wheel" type="continuous">
-        <origin xyz="0.155 0.0722643 0.05" rpy="3.14159 -1.5708 0" />
+        <origin xyz="-0.155 0.0722643 0.05" rpy="3.14159 -1.5708 0" />
         <parent link="body" />
         <child link="right_wheel" />
@@ -167,5 +167,5 @@
     <link name="sensor_laser">
         <visual>
-            <origin xyz="0 -0.125 0.56" rpy="3.14159 -0 0" />
+            <origin xyz="0 -0.125 0.56" rpy="3.14159 0 0" />
             <geometry>
                 <mesh filename="package://deliverybot/urdf/meshes/sensor_laser.stl"/>
@@ -176,5 +176,5 @@
         </visual>
         <collision>
-            <origin xyz="0 -0.125 0.56" rpy="3.14159 -0 0" />
+            <origin xyz="0 -0.125 0.56" rpy="3.14159 0 0" />
             <geometry>
                 <mesh filename="package://deliverybot/urdf/meshes/sensor_laser.stl"/>
@@ -191,5 +191,5 @@
     </link>
     <joint name="joint_laser_sensor" type="fixed">
-        <origin xyz="-5.55112e-17 -0.127736 0.51" rpy="3.14159 -0 0" />
+        <origin xyz="-5.55112e-17 -0.127736 0.535" rpy="0 0 3.14159" />
         <parent link="body" />
         <child link="sensor_laser" />

Commit message: navigation and urdf overhaul

File: deliverybot/urdf/dbot_laser.xacro (robot description, xacro)
@@ -59,8 +59,8 @@
     </link>
     <joint name="joint_left_wheel" type="continuous">
-        <origin xyz="0.155 0.0722643 0.05" rpy="3.14159 -1.5708 0" />
+        <origin xyz="0.155 0.0722643 0.05" rpy="0 -1.5708 0" /> <!-- rpy="-1.5708" -->
         <parent link="body" />
         <child link="left_wheel" />
-        <axis xyz="0 0 1"/>
+        <axis xyz="0 0 -1"/>
         <limit effort="1" velocity="20" />
         <joint_properties friction="0.0"/>
@@ -92,8 +92,8 @@
     </link>
     <joint name="joint_right_wheel" type="continuous">
-        <origin xyz="-0.155 0.0722643 0.05" rpy="3.14159 -1.5708 0" />
+        <origin xyz="-0.155 0.0722643 0.05" rpy="0 -1.5708 0" /> <!-- rpy="-1.5708" -->
         <parent link="body" />
         <child link="right_wheel" />
-        <axis xyz="0 0 1"/>
+        <axis xyz="0 0 -1"/>
         <limit effort="1" velocity="20" />
         <joint_properties friction="0.0"/>

Commit message: Fixed navigation. It finally worksgit add .!

File: deliverybot/urdf/dbot_laser.xacro (robot description, xacro)
@@ -6,5 +6,5 @@
         <parent link="base_link"/>
         <child link="body" />
-        <origin xyz="0 0 0" rpy="0 0 3.141" />
+        <origin xyz="0 0 0" rpy="0 0 1.5707" />
     </joint>
     <link name="body">
