Commit message: Elevator package created with a working custom controller

File: elevator_control/urdf/elevator/elevator.urdf (robot description, URDF)
Before this commit: robot elevator, 11 links, 10 joints
Links:
- link car: geometry collision mesh filename=package://elevator_control/urdf/elevator/car.dae; visual mesh filename=package://elevator_control/urdf/elevator/car.dae
- link car_door_left: geometry collision mesh filename=package://elevator_control/urdf/elevator/car_door_left.dae; visual mesh filename=package://elevator_control/urdf/elevator/car_door_left.dae
- link car_door_right: geometry collision mesh filename=package://elevator_control/urdf/elevator/car_door_right.dae; visual mesh filename=package://elevator_control/urdf/elevator/car_door_right.dae
- link first_door_left: geometry collision mesh filename=package://elevator_control/urdf/elevator/first_door_left.dae; visual mesh filename=package://elevator_control/urdf/elevator/first_door_left.dae
- link first_door_right: geometry collision mesh filename=package://elevator_control/urdf/elevator/first_door_right.d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; visual mesh filename=package://elevator_control/urdf/elevator/first_door_right.d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
- link lobby_door_left: geometry collision mesh filename=package://elevator_control/urdf/elevator/lobby_door_left.dae; visual mesh filename=package://elevator_control/urdf/elevator/lobby_door_left.dae
- link lobby_door_right: geometry collision mesh filename=package://elevator_control/urdf/elevator/lobby_door_right.d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; visual mesh filename=package://elevator_control/urdf/elevator/lobby_door_right.d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
- link second_door_left: geometry collision mesh filename=package://elevator_control/urdf/elevator/second_door_left.d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; visual mesh filename=package://elevator_control/urdf/elevator/second_door_left.d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
- link second_door_right: geometry collision mesh filename=package://elevator_control/urdf/elevator/second_door_right.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; visual mesh filename=package://elevator_control/urdf/elevator/second_door_right.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
- link shaft: geometry collision mesh filename=package://elevator_control/urdf/elevator/shaft.dae; visual mesh filename=package://elevator_control/urdf/elevator/shaft.dae
Joints:
- joint floor: limit lower=0.0 upper=8.0 effort=100000 velocity=0.5 -> lower=0.0 upper=8.0 effort=10000 velocity=0.5
