Commit message: elevator working with no gravity. Had to remove gravity for doors too.

File: elevator_control/models/elevator/elevator.urdf (robot description, URDF)
Before this commit: robot elevator, 11 links, 10 joints
Links:
- link car: geometry collision mesh filename=package://elevator_control/models/elevator/car.dae; visual mesh filename=package://elevator_control/models/elevator/car.dae
- link car_door_left: geometry collision mesh filename=package://elevator_control/models/elevator/car_door_left.dae; visual mesh filename=package://elevator_control/models/elevator/car_door_left.dae
- link car_door_right: geometry collision mesh filename=package://elevator_control/models/elevator/car_door_right.d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; visual mesh filename=package://elevator_control/models/elevator/car_door_right.d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
- link first_door_left: geometry collision mesh filename=package://elevator_control/models/elevator/first_door_left.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; visual mesh filename=package://elevator_control/models/elevator/first_door_left.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
- link first_door_right: geometry collision mesh filename=package://elevator_control/models/elevator/first_door_right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; visual mesh filename=package://elevator_control/models/elevator/first_door_right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
- link lobby_door_left: geometry collision mesh filename=package://elevator_control/models/elevator/lobby_door_left.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; visual mesh filename=package://elevator_control/models/elevator/lobby_door_left.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
- link lobby_door_right: geometry collision mesh filename=package://elevator_control/models/elevator/lobby_door_right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; visual mesh filename=package://elevator_control/models/elevator/lobby_door_right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
- link second_door_left: geometry collision mesh filename=package://elevator_control/models/elevator/second_door_left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; visual mesh filename=package://elevator_control/models/elevator/second_door_left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
- link second_door_right: geometry collision mesh filename=package://elevator_control/models/elevator/second_door_righ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; visual mesh filename=package://elevator_control/models/elevator/second_door_righ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
- link shaft: geometry collision mesh filename=package://elevator_control/models/elevator/shaft.dae; visual mesh filename=package://elevator_control/models/elevator/shaft.dae
