Commit message: Added wingA with new elevator. Have to add option to change floor height.

File: elevator_control/models/wingA_elevator/elevator.urdf (robot description, URDF)
Before this commit: robot elevator, 11 links, 10 joints
Links:
- link car: geometry collision mesh filename=package://elevator_control/models/wingA_elevator/car.dae; visual mesh filename=package://elevator_control/models/wingA_elevator/car.dae
- link car_door_left: geometry collision mesh filename=package://elevator_control/models/wingA_elevator/car_door_l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; visual mesh filename=package://elevator_control/models/wingA_elevator/car_door_l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
- link car_door_right: geometry collision mesh filename=package://elevator_control/models/wingA_elevator/car_door_r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; visual mesh filename=package://elevator_control/models/wingA_elevator/car_door_r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
- link first_door_left: geometry collision mesh filename=package://elevator_control/models/wingA_elevator/first_door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; visual mesh filename=package://elevator_control/models/wingA_elevator/first_door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
- link first_door_right: geometry collision mesh filename=package://elevator_control/models/wingA_elevator/first_door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; visual mesh filename=package://elevator_control/models/wingA_elevator/first_door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
- link lobby_door_left: geometry collision mesh filename=package://elevator_control/models/wingA_elevator/lobby_door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; visual mesh filename=package://elevator_control/models/wingA_elevator/lobby_door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
- link lobby_door_right: geometry collision mesh filename=package://elevator_control/models/wingA_elevator/lobby_door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; visual mesh filename=package://elevator_control/models/wingA_elevator/lobby_door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
- link second_door_left: geometry collision mesh filename=package://elevator_control/models/wingA_elevator/second_doo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; visual mesh filename=package://elevator_control/models/wingA_elevator/second_doo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
- link second_door_right: geometry collision mesh filename=package://elevator_control/models/wingA_elevator/second_doo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; visual mesh filename=package://elevator_control/models/wingA_elevator/second_doo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
- link shaft: geometry collision mesh filename=package://elevator_control/models/wingA_elevator/shaft.dae; visual mesh filename=package://elevator_control/models/wingA_elevator/shaft.dae
