Commit message: Update elevator model, add new simulation world
Signed-off-by: Ammaar Solkar <asketch8@gmail.com>

File: elevator/elevator_description/models/building_elevator/elevator.urdf (robot description, URDF)
Before this commit: robot elevator, 11 links, 10 joints
Links:
- link car: mass 100 -> 1000
