Commit message: Inferno world working

File: deliverybot/deliverybot_description/urdf/dbot.xacro (robot description, xacro)
@@ -125,9 +125,9 @@
     </link>
     <joint name="joint_castor" type="fixed">
-        <origin xyz="-5.55112e-17 -0.127736 -0.025" rpy="0 -0 0" />
+        <origin xyz="-5.55112e-17 -0.127736 -0.025" rpy="0 0 0" />
         <parent link="body" />
         <child link="castor" />
         <axis xyz="0 0 1"/>
-        <limit effort="1" velocity="20" />
+        <limit effort="10000000" velocity="20000" />
         <joint_properties friction="0.0"/>
     </joint>

File: elevator/elevator_description/models/building_elevator/elevator.urdf (robot description, URDF)
Before this commit: robot elevator, 11 links, 10 joints
Links:
- link car: mass 1000 -> 500
Joints:
- joint floor: limit lower=0.0 upper=8.0 effort=10000 velocity=0.5 -> lower=0.0 upper=8.0 effort=10000 velocity=1.0

Commit message: Added 3 new cameras

File: deliverybot/deliverybot_description/urdf/dbot.xacro (robot description, xacro)
@@ -199,7 +199,8 @@
         <joint_properties friction="0.0"/>
     </joint>
+<!-- Lidar -->
 <!-- Kinect -->
     <link name="kinect">
-        <visual>
+        <!-- <visual>
             <geometry>
                 <box size="0.02 0.02 0.02"></box>
@@ -211,6 +212,5 @@
             </geometry>
         </collision>
-        <!-- TODO -->
-        <!-- Add Inertial Element -->
+        Add Inertial Element -->
     </link>
     <joint name="joint_kinect" type="fixed">
@@ -225,4 +225,5 @@
     </joint>
     <link name="kinect_frame_optical"/>
+<!-- Kinect -->
 <!-- Pusher -->
     <link name="pusher">
@@ -252,3 +253,31 @@
         <limit effort="1000" lower="0" upper="0.24" velocity="0.5"/>
     </joint>
+<!-- Pusher -->
+<!-- Upper Camera -->
+  <joint name="upper_camera_joint" type="fixed">
+    <axis xyz="0 1 0" />
+    <origin xyz="-5.55112e-17 -0.127736 0.55" rpy="0 -0.2617 -1.5707" />
+    <parent link="body"/>
+    <child link="upper_camera_link"/>
+  </joint>
+  <link name="upper_camera_link" />
+<!-- Upper Camera -->
+<!-- Right Camera -->
+  <joint name="right_camera_joint" type="fixed">
+    <axis xyz="0 1 0" />
+    <origin xyz="-0.15 0 0.45" rpy="0 0 3.1415" />
+    <parent link="body"/>
+    <child link="right_camera_link"/>
+  </joint>
+  <link name="right_camera_link" />
+<!-- Right Camera -->
+<!-- Left Camera -->
+  <joint name="left_camera_joint" type="fixed">
+    <axis xyz="0 1 0" />
+    <origin xyz="0.15 0 0.45" rpy="0 0 0" />
+    <parent link="body"/>
+    <child link="left_camera_link"/>
+  </joint>
+  <link name="left_camera_link" />
+<!-- Left Camera -->
 </robot>

Commit message: Update deliverybot meshes

File: deliverybot/deliverybot_description/urdf/dbot.xacro (robot description, xacro)
@@ -12,5 +12,5 @@
             <origin xyz="-5.55112e-17 -0.00273569 -0.05" rpy="0 0 0" />
             <geometry>
-                <mesh filename="package://deliverybot_description/urdf/meshes/body.stl"/>
+                <mesh filename="package://deliverybot_description/urdf/meshes/body.dae"/>
             </geometry>
             <material name="body_material">
@@ -21,5 +21,5 @@
             <origin xyz="-5.55112e-17 -0.00273569 -0.05" rpy="0 0 0" />
             <geometry>
-                <mesh filename="package://deliverybot_description/urdf/meshes/body.stl"/>
+                <mesh filename="package://deliverybot_description/urdf/meshes/body.dae"/>
             </geometry>
             <material name="body_material">
@@ -37,5 +37,5 @@
             <origin xyz="-0.075 -0.1 0.155" rpy="-1.5708 -1.5708 0" />
             <geometry>
-                <mesh filename="package://deliverybot_description/urdf/meshes/left_wheel.stl"/>
+                <mesh filename="package://deliverybot_description/urdf/meshes/left_wheel.dae"/>
             </geometry>
             <material name="left_wheel_material">
@@ -46,5 +46,5 @@
             <origin xyz="-0.075 -0.1 0.155" rpy="-1.5708 -1.5708 0" />
             <geometry>
-                <mesh filename="package://deliverybot_description/urdf/meshes/left_wheel.stl"/>
+                <mesh filename="package://deliverybot_description/urdf/meshes/left_wheel.dae"/>
             </geometry>
             <material name="left_wheel_material">
@@ -70,5 +70,5 @@
             <origin xyz="-0.075 -0.1 -0.155" rpy="-1.5708 -1.5708 0" />
             <geometry>
-                <mesh filename="package://deliverybot_description/urdf/meshes/right_wheel.stl"/>
+                <mesh filename="package://deliverybot_description/urdf/meshes/right_wheel.dae"/>
             </geometry>
             <material name="left_wheel_material">
@@ -79,5 +79,5 @@
             <origin xyz="-0.075 -0.1 -0.155" rpy="-1.5708 -1.5708 0" />
             <geometry>
-                <mesh filename="package://deliverybot_description/urdf/meshes/right_wheel.stl"/>
+                <mesh filename="package://deliverybot_description/urdf/meshes/right_wheel.dae"/>
             </geometry>
             <material name="right_wheel_material">
@@ -103,5 +103,5 @@
             <origin xyz="0 0.125 -0.025" rpy="0 -0 0" />
             <geometry>
-                <mesh filename="package://deliverybot_description/urdf/meshes/castor.stl"/>
+                <mesh filename="package://deliverybot_description/urdf/meshes/castor.dae"/>
             </geometry>
             <material name="castor_material">
@@ -112,5 +112,5 @@
             <origin xyz="0 0.125 -0.025" rpy="0 -0 0" />
             <geometry>
-                <mesh filename="package://deliverybot_description/urdf/meshes/castor.stl"/>
+                <mesh filename="package://deliverybot_description/urdf/meshes/castor.dae"/>
             </geometry>
             <material name="castor_material">
@@ -136,5 +136,5 @@
             <origin xyz="0.127 -0.205 -0.145" rpy="-1.5708 -1.5708 0" />
             <geometry>
-                <mesh filename="package://deliverybot_description/urdf/meshes/door.stl"/>
+                <mesh filename="package://deliverybot_description/urdf/meshes/door.dae"/>
             </geometry>
             <material name="door_material">
@@ -145,5 +145,5 @@
             <origin xyz="0.127 -0.205 -0.145" rpy="-1.5708 -1.5708 0" />
             <geometry>
-                <mesh filename="package://deliverybot_description/urdf/meshes/door.stl"/>
+                <mesh filename="package://deliverybot_description/urdf/meshes/door.dae"/>
             </geometry>
             <material name="door_material">
@@ -170,5 +170,5 @@
             <origin xyz="0 -0.125 0.56" rpy="3.14159 0 0" />
             <geometry>
-                <mesh filename="package://deliverybot_description/urdf/meshes/sensor_laser.stl"/>
+                <mesh filename="package://deliverybot_description/urdf/meshes/sensor_laser.dae"/>
             </geometry>
             <material name="sensor_laser_material">
@@ -179,5 +179,5 @@
             <origin xyz="0 -0.125 0.56" rpy="3.14159 0 0" />
             <geometry>
-                <mesh filename="package://deliverybot_description/urdf/meshes/sensor_laser.stl"/>
+                <mesh filename="package://deliverybot_description/urdf/meshes/sensor_laser.dae"/>
             </geometry>
             <material name="sensor_laser_material">
